File: self-tuning-buck-converter/design/PCBs/Breakouts/50mOhm_Shunt/50mOhm_Shunt.sch (KiCad schematic (older format))
At the start: 5 parts, among them J1 Input +, J2 Kelvin +, J3 Input -, J4 Kelvin -

Commit message: update breakout PCB's for the 50mO and 60mO resistors. Ordered the missing parts
Parts:
- J1, J2, J3, J4: footprint Connector_PinHeader_1.00mm:PinHeader_1x01_P1.00mm_Vertical -> Connector_PinHeader_2.54mm:PinHeader_1x01_P2.54mm_Vertical
Changed lines of the file:
@@
 F 0 "J3" H 2550 1650 50  0000 R CNN
 F 1 "Input -" H 2850 1550 50  0000 R CNN
-F 2 "Connector_PinHeader_1.00mm:PinHeader_1x01_P1.00mm_Vertical" H 2500 1450 50  0001 C CNN
+F 2 "Connector_PinHeader_2.54mm:PinHeader_1x01_P2.54mm_Vertical" H 2500 1450 50  0001 C CNN
 F 3 "~" H 2500 1450 50  0001 C CNN
 	1    2500 1450
@@
 F 0 "J1" H 1208 1631 50  0000 C CNN
 F 1 "Input +" H 1208 1540 50  0000 C CNN
-F 2 "Connector_PinHeader_1.00mm:PinHeader_1x01_P1.00mm_Vertical" H 1100 1450 50  0001 C CNN
+F 2 "Connector_PinHeader_2.54mm:PinHeader_1x01_P2.54mm_Vertical" H 1100 1450 50  0001 C CNN
 F 3 "~" H 1100 1450 50  0001 C CNN
 	1    1100 1450
@@
 F 0 "J2" H 1208 1981 50  0000 C CNN
 F 1 "Kelvin +" H 1208 1890 50  0000 C CNN
-F 2 "Connector_PinHeader_1.00mm:PinHeader_1x01_P1.00mm_Vertical" H 1100 1800 50  0001 C CNN
+F 2 "Connector_PinHeader_2.54mm:PinHeader_1x01_P2.54mm_Vertical" H 1100 1800 50  0001 C CNN
 F 3 "~" H 1100 1800 50  0001 C CNN
 	1    1100 1800
@@
 F 0 "J4" H 2550 2000 50  0000 R CNN
 F 1 "Kelvin -" H 2850 1900 50  0000 R CNN
-F 2 "Connector_PinHeader_1.00mm:PinHeader_1x01_P1.00mm_Vertical" H 2500 1800 50  0001 C CNN
+F 2 "Connector_PinHeader_2.54mm:PinHeader_1x01_P2.54mm_Vertical" H 2500 1800 50  0001 C CNN
 F 3 "~" H 2500 1800 50  0001 C CNN
 	1    2500 1800
