File: self-tuning-buck-converter/PCBs/Breakouts/60mOhm_Shunt/60mOhm_Shunt.kicad_pcb (KiCad board)
At the start: 2 copper layers, 15.7 x 7.6 mm, 5 parts, among them J1 Input +, J2 Kelvin +, J3 Input -, J4 Kelvin -

Commit message: began PCB design for entire buck converter
Other:
- board text added: "60m"
- board text removed: "60 mOhms"
